Commit message: task controller bug fixing...

File: dyros_jet_description/robots/dyros_jet_robot.urdf (robot description, URDF)
Before this commit: robot dyros_jet_robot, 30 links, 29 joints
Links:
- removed link L_AnckleRoll_Link
- removed link R_AncklePitch_Link
- removed link R_AnckleRoll_Link
- added link L_AnkleRoll_Link, mass 1.297; collision mesh filename=package://dyros_jet_description/meshes/L_AnkleRoll_Link.stl; visual mesh filename=package://dyros_jet_description/meshes/L_AnkleRoll_Link.stl
- added link R_AnklePitch_Link, mass 1.0349; collision mesh filename=package://dyros_jet_description/meshes/R_AnklePitch_Link.stl; visual mesh filename=package://dyros_jet_description/meshes/R_AnklePitch_Link.stl
- added link R_AnkleRoll_Link, mass 1.297; collision mesh filename=package://dyros_jet_description/meshes/R_AnkleRoll_Link.stl; visual mesh filename=package://dyros_jet_description/meshes/R_AnkleRoll_Link.stl
Joints:
- removed joint L_AnckleRoll
- removed joint R_AncklePitch
- removed joint R_AnckleRoll
- added joint L_AnkleRoll: type revolute, parent L_AnklePitch_Link, child L_AnkleRoll_Link, origin xyz=0 0 0 rpy=0 0 0, axis 1 0 0, limit lower=-3.14 upper=3.14 effort=30 velocity=1
- added joint R_AnklePitch: type revolute, parent R_KneePitch_Link, child R_AnklePitch_Link, origin xyz=0.06 -0.00485 -0.368 rpy=-1.2837E-16 -4.4988E-16 -3.5523E-16, axis 0 -1 0, limit lower=-3.14 upper=3.14 effort=30 velocity=1
- added joint R_AnkleRoll: type revolute, parent R_AnklePitch_Link, child R_AnkleRoll_Link, origin xyz=0 0 0 rpy=0 9.8608E-32 1.8489E-32, axis 1 0 0, limit lower=-3.14 upper=3.14 effort=30 velocity=1

Commit message: virtual joint add

File: dyros_jet_description/robots/dyros_jet_robot.urdf (robot description, URDF)
Before this commit: robot dyros_jet_robot, 30 links, 29 joints
Joints:
- joint virtual: limit lower=-2.2 upper=0.7 effort=30 velocity=1.0 -> effort=30 velocity=1.0; type fixed -> floating

Commit message: urdf changed

File: dyros_jet_description/robots/dyros_jet_robot.urdf (robot description, URDF)
Before this commit: robot dyros_jet_robot, 30 links, 29 joints
Joints:
- joint L_AnklePitch: origin xyz=0.06 0.00485 -0.36794 rpy=0 0 0 -> xyz=0.06 0.00485 -0.368 rpy=0 0 0
- joint L_HipRoll: origin xyz=-0.0059 -0.00026292 -0.1349 rpy=0 0 0 -> xyz=-0.0059 0 -0.1349 rpy=0 0 0
- joint L_HipYaw: origin xyz=0 0.10526 0 rpy=0 0 0 -> xyz=0 0.105 0 rpy=0 0 0
- joint L_KneePitch: origin xyz=0.1515 -0.01075 -0.33906 rpy=0 0 0 -> xyz=0.1515 -0.01075 -0.339 rpy=0 0 0
- joint R_AnklePitch: origin xyz=0.06 -0.00485 -0.368 rpy=-1.2837E-16 -4.4988E-16 -3.5523E-16 -> xyz=0.06 -0.00485 -0.368 rpy=0 0 0
- joint R_AnkleRoll: origin xyz=0 0 0 rpy=0 9.8608E-32 1.8489E-32 -> xyz=0 0 0 rpy=0 0 0
- joint R_HipPitch: origin xyz=0 0 0 rpy=3.4694E-18 7.7037E-34 -3.6352E-33 -> xyz=0 0 0 rpy=0 0 0
- joint R_HipRoll: origin xyz=-0.0059 0 -0.1349 rpy=-0.018707 -6.6457E-18 -5.7725E-16 -> xyz=-0.0059 0 -0.1349 rpy=0 0 0
- joint R_KneePitch: origin xyz=0.1515 0.01075 -0.339 rpy=-1.7347E-17 3.0195E-18 5.7728E-16 -> xyz=0.1515 0.01075 -0.339 rpy=0 0 0

Commit message: revise urdf & stl

File: dyros_jet_description/robots/dyros_jet_robot.urdf (robot description, URDF)
Before this commit: robot dyros_jet_robot, 30 links, 29 joints
Links:
- link L_AnklePitch_Link: mass 1.0349 -> 1.18450; geometry collision mesh filename=package://dyros_jet_description/meshes/left_ankle_pitch.stl; visual mesh filename=package://dyros_jet_description/meshes/left_ankle_pitch.stl
- link L_AnkleRoll_Link: mass 1.297 -> 1.42541; geometry collision mesh filename=package://dyros_jet_description/meshes/ankle_roll.stl; visual mesh filename=package://dyros_jet_description/meshes/ankle_roll.stl
- link L_ElbowRoll_Link: mass 0.83343 -> 0.83342
- link L_HandYaw_Link: mass 1.206 -> 1.20640
- link L_HipPitch_Link: mass 3.2021 -> 3.28269; geometry collision mesh filename=package://dyros_jet_description/meshes/hip_pitch.stl; visual mesh filename=package://dyros_jet_description/meshes/hip_pitch.stl
- link L_HipRoll_Link: mass 1.023 -> 1.16907; geometry collision mesh filename=package://dyros_jet_description/meshes/hip_roll.stl; visual mesh filename=package://dyros_jet_description/meshes/hip_roll.stl
- link L_HipYaw_Link: mass 1.495 -> 1.54216; geometry collision mesh filename=package://dyros_jet_description/meshes/hip_yaw.stl; visual mesh filename=package://dyros_jet_description/meshes/hip_yaw.stl
- link L_KneePitch_Link: mass 2.0241 -> 2.04524; geometry collision mesh filename=package://dyros_jet_description/meshes/left_shin.stl; visual mesh filename=package://dyros_jet_description/meshes/left_shin.stl
- link L_ShoulderPitch_Link: mass 0.92826 -> 0.92796
- link L_ShoulderRoll_Link: mass 0.37361 -> 0.11240
- link L_ShoulderYaw_Link: mass 1.7512 -> 1.75149
- link L_WristRoll_Link: mass 0.0695 -> 0.07856
- link L_WristYaw_Link: mass 0.52387 -> 0.52391
- link R_AnklePitch_Link: mass 1.0349 -> 1.18450; geometry collision mesh filename=package://dyros_jet_description/meshes/right_ankle_pitch.stl; visual mesh filename=package://dyros_jet_description/meshes/right_ankle_pitch.stl
- link R_AnkleRoll_Link: mass 1.297 -> 1.42541; geometry collision mesh filename=package://dyros_jet_description/meshes/ankle_roll.stl; visual mesh filename=package://dyros_jet_description/meshes/ankle_roll.stl
- link R_ElbowRoll_Link: mass 0.83343 -> 0.83342
- link R_HandYaw_Link: mass 1.206 -> 1.20640
- link R_HipPitch_Link: mass 3.2021 -> 3.28269; geometry collision mesh filename=package://dyros_jet_description/meshes/hip_pitch.stl; visual mesh filename=package://dyros_jet_description/meshes/hip_pitch.stl
- link R_HipRoll_Link: mass 1.023 -> 1.16907; geometry collision mesh filename=package://dyros_jet_description/meshes/hip_roll.stl; visual mesh filename=package://dyros_jet_description/meshes/hip_roll.stl
- link R_HipYaw_Link: mass 1.495 -> 1.54216; geometry collision mesh filename=package://dyros_jet_description/meshes/hip_yaw.stl; visual mesh filename=package://dyros_jet_description/meshes/hip_yaw.stl
- link R_KneePitch_Link: mass 2.0241 -> 2.04524; geometry collision mesh filename=package://dyros_jet_description/meshes/right_shin.stl; visual mesh filename=package://dyros_jet_description/meshes/right_shin.stl
- link R_ShoulderPitch_Link: mass 0.92826 -> 0.92796
- link R_ShoulderRoll_Link: mass 0.37361 -> 0.11240
- link R_ShoulderYaw_Link: mass 1.7512 -> 1.75149
- link R_WristRoll_Link: mass 0.0695 -> 0.07856
- link R_WristYaw_Link: mass 0.52387 -> 0.52391
- link WaistPitch_Link: mass 0.17684 -> 0.18235
- link WaistYaw_Link: mass 10.78 -> 14.09938
- link base_link: mass 1.9994 -> 3.90994
Joints:
- joint L_AnklePitch: origin xyz=0.06 0.00485 -0.368 rpy=0 0 0 -> xyz=0.06 0 -0.368 rpy=0 0 0
- joint L_HipRoll: origin xyz=-0.0059 0 -0.1349 rpy=0 0 0 -> xyz=0 0 0 rpy=0 0 0
- joint L_HipYaw: origin xyz=0 0.105 0 rpy=0 0 0 -> xyz=0 0.105 -0.11190 rpy=0 0 0
- joint L_KneePitch: origin xyz=0.1515 -0.01075 -0.339 rpy=0 0 0 -> xyz=0.1515 0 ?0.339 rpy=0 0 0
- joint R_AnklePitch: origin xyz=0.06 -0.00485 -0.368 rpy=0 0 0 -> xyz=0.06 0 -0.368 rpy=0 0 0
- joint R_HipRoll: origin xyz=-0.0059 0 -0.1349 rpy=0 0 0 -> xyz=0 0 0 rpy=0 0 0
- joint R_HipYaw: origin xyz=0 -0.105 0 rpy=0 0 0 -> xyz=0 -0.105 -0.11190 rpy=0 0 0
- joint R_KneePitch: origin xyz=0.1515 0.01075 -0.339 rpy=0 0 0 -> xyz=0.1515 0 ?0.339 rpy=0 0 0

Commit message: urdf

File: dyros_jet_description/robots/dyros_jet_robot.urdf (robot description, URDF)
Before this commit: robot dyros_jet_robot, 30 links, 29 joints
Joints:
- joint L_KneePitch: origin xyz=0.1515 0 ?0.339 rpy=0 0 0 -> xyz=0.1515 0 0.339 rpy=0 0 0
- joint R_KneePitch: origin xyz=0.1515 0 ?0.339 rpy=0 0 0 -> xyz=0.1515 0 0.339 rpy=0 0 0

Commit message: newscene

File: dyros_jet_description/robots/dyros_jet_robot.urdf (robot description, URDF)
Before this commit: robot dyros_jet_robot, 30 links, 29 joints
Links:
- removed link world
Joints:
- removed joint virtual
- joint L_KneePitch: origin xyz=0.1515 0 0.339 rpy=0 0 0 -> xyz=0.1515 0 -0.339 rpy=0 0 0
- joint R_KneePitch: origin xyz=0.1515 0 0.339 rpy=0 0 0 -> xyz=0.1515 0 -0.339 rpy=0 0 0

Commit message: virtual joint inserted

File: dyros_jet_description/robots/dyros_jet_robot.urdf (robot description, URDF)
Before this commit: robot dyros_jet_robot, 29 links, 28 joints
Links:
- added link world
Joints:
- added joint virtual: type floating, parent world, child base_link, origin xyz=0 0 0 rpy=0 0 0, limit lower=-3.14 upper=3.14 effort=30 velocity=1.0

Commit message: exp

File: dyros_jet_description/robots/dyros_jet_robot.urdf (robot description, URDF)
Before this commit: robot dyros_jet_robot, 30 links, 29 joints
Links:
- link R_HandYaw_Link: mass 1.20640 -> 0.90640

Commit message: moveit edit

File: dyros_jet_description/robots/dyros_jet_robot.urdf (robot description, URDF)
Before this commit: robot dyros_jet_robot, 29 links, 28 joints
Links:
- link R_HandYaw_Link: geometry collision mesh filename=package://dyros_jet_description/meshes/R_HandYaw_new.stl; visual mesh filename=package://dyros_jet_description/meshes/R_HandYaw_new.stl
Joints:
- joint L_ElbowRoll: limit lower=-3.14 upper=3.14 effort=30 velocity=1 -> lower=-2.8 upper=0.3 effort=30 velocity=1
- joint L_ShoulderRoll: limit lower=-3.14 upper=3.14 effort=30 velocity=1 -> lower=-2.1 upper=-0.2 effort=30 velocity=1
- joint R_ElbowRoll: limit lower=-3.14 upper=3.14 effort=30 velocity=1 -> lower=-0.3 upper=2.8 effort=30 velocity=1
- joint R_ShoulderRoll: limit lower=-3.14 upper=3.14 effort=30 velocity=1 -> lower=0.2 upper=2.1 effort=30 velocity=1
- joint R_WristRoll: limit lower=-3.14 upper=3.14 effort=30 velocity=1 -> lower=-1.9 upper=1.9 effort=30 velocity=1

Commit message: urdf torso backpack added

File: dyros_jet_description/robots/dyros_jet_robot.urdf (robot description, URDF)
Before this commit: robot dyros_jet_robot, 29 links, 28 joints
Links:
- link WaistYaw_Link: geometry collision box size=0.09 0.265 0.225; collision mesh filename=package://dyros_jet_description/meshes/WaistYaw_Link.stl

Commit message: when it walk, left foot hit the ground

File: dyros_jet_description/robots/dyros_jet_robot.urdf (robot description, URDF)
Before this commit: robot dyros_jet_robot, 30 links, 29 joints
Links:
- link R_HandYaw_Link: mass 0.90640 -> 0.80640

Commit message: com jacobian added

File: dyros_jet_description/robots/dyros_jet_robot.urdf (robot description, URDF)
Before this commit: robot dyros_jet_robot, 30 links, 29 joints
Links:
- link R_HandYaw_Link: mass 0.80640 -> 1.20640
